Commit message: Rename 'taurob_robot_description' to 'taurob_tracker_description'.

File: taurob_tracker_description/urdf/tracker_chassis.urdf.xacro (robot description, xacro)
@@ -48,5 +48,5 @@
         <origin xyz="0.0 0.0 0.0" rpy="0 0 0" />
         <geometry>
-          <mesh filename="package://taurob_robot_description/meshes/tracker/tracker_chassis.dae"/>
+          <mesh filename="package://taurob_tracker_description/meshes/tracker/tracker_chassis.dae"/>
         </geometry>
       </visual>
