Commit message: Clean up URDF models.

File: taurob_tracker_description/urdf/tracker.urdf.xacro (robot description, xacro)
@@ -1,5 +1,4 @@
 <?xml version="1.0"?>
-<robot name="taurob_tracker"
-  xmlns:xacro="http://www.ros.org/wiki/xacro">
+<robot xmlns:xacro="http://www.ros.org/wiki/xacro" name="taurob_tracker">
   <xacro:property name="flipper_offset_x" value="0.205"/>
   <xacro:property name="flipper_offset_y" value="0.15"/>

File: taurob_tracker_description/urdf/tracker_arm.urdf.xacro (robot description, xacro)
@@ -1,177 +1,162 @@
 <?xml version="1.0"?>
-<robot
-    xmlns:sensor="http://playerstage.sourceforge.net/gazebo/xmlschema/#sensor"
-    xmlns:controller="http://playerstage.sourceforge.net/gazebo/xmlschema/#controller"
-    xmlns:interface="http://playerstage.sourceforge.net/gazebo/xmlschema/#interface">
-    <xacro:property name="base_size_x" value="0.92" />
-    <xacro:property name="base_size_y" value="0.24" />
-    <xacro:property name="base_size_z" value="0.34" />
-    <xacro:property name="M_PI" value="3.14159265359" />
-    <xacro:macro name="taurob_arm_macro" params="parent *origin">
-	<joint name="arm_joint_0" type="revolute">
-		<xacro:insert_block name="origin"/>
-		<axis xyz="0 0 1"/>
-		<limit lower="${-180 * M_PI / 180}" upper="${180 * M_PI / 180}"
-		     effort="1000" velocity="${1.0 * 110 * M_PI / 180}" />
-		<!--        <safety_controller soft_lower_limit="${-168 * M_PI / 180}"
+<robot xmlns:xacro="http://www.ros.org/wiki/xacro">
+  <xacro:property name="base_size_x" value="0.92"/>
+  <xacro:property name="base_size_y" value="0.24"/>
+  <xacro:property name="base_size_z" value="0.34"/>
+  <xacro:property name="M_PI" value="3.14159265359"/>
+  <xacro:macro name="tracker_arm_macro" params="parent *origin">
+    <joint name="arm_joint_0" type="revolute">
+      <xacro:insert_block name="origin"/>
+      <axis xyz="0 0 1"/>
+      <limit lower="${-180 * M_PI / 180}" upper="${180 * M_PI / 180}" effort="1000" velocity="${1.0 * 110 * M_PI / 180}"/>
+      <!--        <safety_controller soft_lower_limit="${-168 * M_PI / 180}"
 				 soft_upper_limit="${168 * M_PI / 180}"
 				 k_position="${100}"
 				 k_velocity="${2}"/>-->
-		<parent link="${parent}"/>
-		<child link="arm_link_0"/>
-	</joint>
-        <link name="arm_link_0">
-            <inertial>
-                <mass value="1.0" />
-                <origin xyz="0.0 0.0 0.0" rpy="0 0 0" />
-                <inertia ixx="0.005" ixy="0.0" ixz="0.0"
-                         iyy="0.005" iyz="0.0"
-                         izz="0.005" />
-            </inertial>
-            <visual>
-                <origin xyz="0.0 0.0 0.0" rpy="0 0 ${M_PI / 2}" />
-                <geometry>
-                    <mesh filename="package://taurob_arm_description/meshes/tarm_link_0.stl"/>
-                </geometry>
-                <material name="DarkGrey" >
-                    <color rgba="0.8 0.8 0.8 1"/>
-                </material>
-            </visual>
-	    <arm_link_0_collision_geom_marco/>
-        </link>
-	<joint name="arm_joint_1" type="revolute">
-		<origin xyz="-0.052 0.0 0.1" rpy="0 0 0" />
-		<axis xyz="1 0 0"/>
-		<limit lower="${0 * M_PI / 180}" upper="${180 * M_PI / 180}"
-		     effort="1000" velocity="${1.0 * 110 * M_PI / 180}" />
-		<!--        <safety_controller soft_lower_limit="${-168 * M_PI / 180}"
+      <parent link="${parent}"/>
+      <child link="arm_link_0"/>
+    </joint>
+    <link name="arm_link_0">
+      <inertial>
+        <mass value="1.0"/>
+        <origin xyz="0.0 0.0 0.0" rpy="0 0 0"/>
+        <inertia ixx="0.005" ixy="0.0" ixz="0.0" iyy="0.005" iyz="0.0" izz="0.005"/>
+      </inertial>
+      <visual>
+        <origin xyz="0.0 0.0 0.0" rpy="0 0 ${M_PI / 2}"/>
+        <geometry>
+          <mesh filename="package://taurob_tracker_description/meshes/tarm_link_0.stl"/>
+        </geometry>
+        <material name="DarkGrey">
+          <color rgba="0.8 0.8 0.8 1"/>
+        </material>
+      </visual>
+      <arm_link_0_collision_geom_marco/>
+    </link>
+    <joint name="arm_joint_1" type="revolute">
+      <origin xyz="-0.052 0.0 0.1" rpy="0 0 0"/>
+      <axis xyz="1 0 0"/>
+      <limit lower="${0 * M_PI / 180}" upper="${180 * M_PI / 180}" effort="1000" velocity="${1.0 * 110 * M_PI / 180}"/>
+      <!--        <safety_controller soft_lower_limit="${-168 * M_PI / 180}"
 				 soft_upper_limit="${168 * M_PI / 180}"
 				 k_position="${100}"
 				 k_velocity="${2}"/>-->
-		<parent link="arm_link_0"/>
-		<child link="arm_link_1"/>
-	</joint>
-        <link name="arm_link_1">
-            <inertial>
-                <mass value="1.0" />
-                <origin xyz="0.0 0.0 0.0" rpy="0 0 0" />
-                <inertia ixx="0.005" ixy="0.0" ixz="0.0"
-                         iyy="0.005" iyz="0.0"
-                         izz="0.005" />
-            </inertial>
-            <visual>
-                <origin xyz="0.0 0.0 0.0" rpy="0 0 0" />
-                <geometry>
-                    <mesh filename="package://taurob_arm_description/meshes/tarm_link_1.stl"/>
-                </geometry>
-                <material name="DarkGrey" >
-                    <color rgba="0.8 0.8 0.8 1"/>
-                </material>
-            </visual>
-            <arm_link_1_collision_geom_marco/>
-        </link>
-	<joint name="arm_joint_2" type="revolute">
-		<origin xyz="0.003 0.55 0.03" rpy=" 0 0 0" />
-		<axis xyz="-1 0 0"/>
-		<limit lower="${0 * M_PI / 180}" upper="${180 * M_PI / 180}"
-			effort="1000" velocity="${1.0 * 110 * M_PI / 180}" />
-		<!--        <safety_controller soft_lower_limit="${-168 * M_PI / 180}"
+      <parent link="arm_link_0"/>
+      <child link="arm_link_1"/>
+    </joint>
+    <link name="arm_link_1">
+      <inertial>
+        <mass value="1.0"/>
+        <origin xyz="0.0 0.0 0.0" rpy="0 0 0"/>
+        <inertia ixx="0.005" ixy="0.0" ixz="0.0" iyy="0.005" iyz="0.0" izz="0.005"/>
+      </inertial>
+      <visual>
+        <origin xyz="0.0 0.0 0.0" rpy="0 0 0"/>
+        <geometry>
+          <mesh filename="package://taurob_tracker_description/meshes/tarm_link_1.stl"/>
+        </geometry>
+        <material name="DarkGrey">
+          <color rgba="0.8 0.8 0.8 1"/>
+        </material>
+      </visual>
+      <arm_link_1_collision_geom_marco/>
+    </link>
+    <joint name="arm_joint_2" type="revolute">
+      <origin xyz="0.003 0.55 0.03" rpy=" 0 0 0"/>
+      <axis xyz="-1 0 0"/>
+      <limit lower="${0 * M_PI / 180}" upper="${180 * M_PI / 180}" effort="1000" velocity="${1.0 * 110 * M_PI / 180}"/>
+      <!--        <safety_controller soft_lower_limit="${-168 * M_PI / 180}"
 				 soft_upper_limit="${168 * M_PI / 180}"
 				 k_position="${100}"
 				 k_velocity="${2}"/>-->
-		<parent link="arm_link_1"/>
-		<child link="arm_link_2"/>
-	</joint>
-        <link name="arm_link_2">
-            <inertial>
-                <mass value="0.1" />
-                <origin xyz="0.0 0.0 0.0" rpy="0 0 0" />
-                <inertia ixx="0.005" ixy="0.0" ixz="0.0"
-                         iyy="0.005" iyz="0.0"
-                         izz="0.005" />
-            </inertial>
-            <visual>
-                <origin xyz="0.0 0.0 0.0" rpy="0 0 0" />
-                <geometry>
-                    <mesh filename="package://taurob_arm_description/meshes/tarm_link_2.stl"/>
-                </geometry>
-                <material name="DarkGrey" >
-                    <color rgba="0.8 0.8 0.8 1"/>
-                </material>
-            </visual>
-            <arm_link_2_collision_geom_marco/>
-          </link>
-	<joint name="arm_joint_3" type="revolute">
-		<origin xyz="0.096 -0.42 0" rpy=" 0 0 0" />
-		<axis xyz="-1 0 0"/>
-		<limit lower="${-180 * M_PI / 180}" upper="${180 * M_PI / 180}"
-			effort="1000" velocity="${1.0 * 110 * M_PI / 180}" />
-		<!--        <safety_controller soft_lower_limit="${-168 * M_PI / 180}"
+      <parent link="arm_link_1"/>
+      <child link="arm_link_2"/>
+    </joint>
+    <link name="arm_link_2">
+      <inertial>
+        <mass value="0.1"/>
+        <origin xyz="0.0 0.0 0.0" rpy="0 0 0"/>
+        <inertia ixx="0.005" ixy="0.0" ixz="0.0" iyy="0.005" iyz="0.0" izz="0.005"/>
+      </inertial>
+      <visual>
+        <origin xyz="0.0 0.0 0.0" rpy="0 0 0"/>
+        <geometry>
+          <mesh filename="package://taurob_tracker_description/meshes/tarm_link_2.stl"/>
+        </geometry>
+        <material name="DarkGrey">
+          <color rgba="0.8 0.8 0.8 1"/>
+        </material>
+      </visual>
+      <arm_link_2_collision_geom_marco/>
+    </link>
+    <joint name="arm_joint_3" type="revolute">
+      <origin xyz="0.096 -0.42 0" rpy=" 0 0 0"/>
+      <axis xyz="-1 0 0"/>
+      <limit lower="${-180 * M_PI / 180}" upper="${180 * M_PI / 180}" effort="1000" velocity="${1.0 * 110 * M_PI / 180}"/>
+      <!--        <safety_controller soft_lower_limit="${-168 * M_PI / 180}"
 			 soft_upper_limit="${168 * M_PI / 180}"
 			 k_position="${100}"
 			 k_velocity="${2}"/>-->
-		<parent link="arm_link_2"/>
-		<child link="arm_link_3"/>
-	</joint>
-          <link name="arm_link_3">
-            <inertial>
-                <mass value="0.1" />
-                <origin xyz="0.0 0.0 0.0" rpy="0 0 0" />
-                <inertia ixx="0.005" ixy="0.0" ixz="0.0"
-                         iyy="0.005" iyz="0.0"
-                         izz="0.005" />
-            </inertial>
-            <visual>
-                <origin xyz="0.0 0.0 0.0" rpy="0 0 0" />
-                <geometry>
-                    <mesh filename="package://taurob_arm_description/meshes/tarm_link_3.stl"/>
-                </geometry>
-                <material name="DarkGrey" >
-                    <color rgba="0.8 0.8 0.8 1"/>
-                </material>
-            </visual>
-            <arm_link_3_collision_geom_marco/>
-        </link>
-        <!--Needed for simulation-->
-          <transmission name="arm_joint_0_joint_transmssion">
-    <type>transmission_interface/SimpleTransmission</type>
-    <joint name="arm_joint_0">
-      <hardwareInterface>EffortJointInterface</hardwareInterface>
+      <parent link="arm_link_2"/>
+      <child link="arm_link_3"/>
     </joint>
-    <actuator name="arm_joint_0_motor">
-      <hardwareInterface>EffortJointInterface</hardwareInterface>
-      <mechanicalReduction>1</mechanicalReduction>
-    </actuator>
-  </transmission>
-  <transmission name="arm_joint_1_joint_transmssion">
-    <type>transmission_interface/SimpleTransmission</type>
-    <joint name="arm_joint_1">
-      <hardwareInterface>EffortJointInterface</hardwareInterface>
-    </joint>
-    <actuator name="arm_joint_1_motor">
-      <hardwareInterface>EffortJointInterface</hardwareInterface>
-      <mechanicalReduction>1</mechanicalReduction>
-    </actuator>
-  </transmission>
-  <transmission name="arm_joint_2_joint_transmssion">
-    <type>transmission_interface/SimpleTransmission</type>
-    <joint name="arm_joint_2">
-      <hardwareInterface>EffortJointInterface</hardwareInterface>
-    </joint>
-    <actuator name="arm_joint_2_motor">
-      <hardwareInterface>EffortJointInterface</hardwareInterface>
-      <mechanicalReduction>1</mechanicalReduction>
-    </actuator>
-  </transmission>
-  <transmission name="arm_joint_3_joint_transmssion">
-    <type>transmission_interface/SimpleTransmission</type>
-    <joint name="arm_joint_3">
-      <hardwareInterface>EffortJointInterface</hardwareInterface>
-    </joint>
-    <actuator name="arm_joint_3_motor">
-      <hardwareInterface>EffortJointInterface</hardwareInterface>
-      <mechanicalReduction>1</mechanicalReduction>
-    </actuator>
-  </transmission>
+    <link name="arm_link_3">
+      <inertial>
+        <mass value="0.1"/>
+        <origin xyz="0.0 0.0 0.0" rpy="0 0 0"/>
+        <inertia ixx="0.005" ixy="0.0" ixz="0.0" iyy="0.005" iyz="0.0" izz="0.005"/>
+      </inertial>
+      <visual>
+        <origin xyz="0.0 0.0 0.0" rpy="0 0 0"/>
+        <geometry>
+          <mesh filename="package://taurob_tracker_description/meshes/tarm_link_3.stl"/>
+        </geometry>
+        <material name="DarkGrey">
+          <color rgba="0.8 0.8 0.8 1"/>
+        </material>
+      </visual>
+      <arm_link_3_collision_geom_marco/>
+    </link>
+    <!--Needed for simulation-->
+    <transmission name="arm_joint_0_joint_transmssion">
+      <type>transmission_interface/SimpleTransmission</type>
+      <joint name="arm_joint_0">
+        <hardwareInterface>EffortJointInterface</hardwareInterface>
+      </joint>
+      <actuator name="arm_joint_0_motor">
+        <hardwareInterface>EffortJointInterface</hardwareInterface>
+        <mechanicalReduction>1</mechanicalReduction>
+      </actuator>
+    </transmission>
+    <transmission name="arm_joint_1_joint_transmssion">
+      <type>transmission_interface/SimpleTransmission</type>
+      <joint name="arm_joint_1">
+        <hardwareInterface>EffortJointInterface</hardwareInterface>
+      </joint>
+      <actuator name="arm_joint_1_motor">
+        <hardwareInterface>EffortJointInterface</hardwareInterface>
+        <mechanicalReduction>1</mechanicalReduction>
+      </actuator>
+    </transmission>
+    <transmission name="arm_joint_2_joint_transmssion">
+      <type>transmission_interface/SimpleTransmission</type>
+      <joint name="arm_joint_2">
+        <hardwareInterface>EffortJointInterface</hardwareInterface>
+      </joint>
+      <actuator name="arm_joint_2_motor">
+        <hardwareInterface>EffortJointInterface</hardwareInterface>
+        <mechanicalReduction>1</mechanicalReduction>
+      </actuator>
+    </transmission>
+    <transmission name="arm_joint_3_joint_transmssion">
+      <type>transmission_interface/SimpleTransmission</type>
+      <joint name="arm_joint_3">
+        <hardwareInterface>EffortJointInterface</hardwareInterface>
+      </joint>
+      <actuator name="arm_joint_3_motor">
+        <hardwareInterface>EffortJointInterface</hardwareInterface>
+        <mechanicalReduction>1</mechanicalReduction>
+      </actuator>
+    </transmission>
     <gazebo reference="arm_link_0">
       <material>Gazebo/Grey</material>
@@ -186,4 +171,4 @@
       <material>Gazebo/Grey</material>
     </gazebo>
-    </xacro:macro>
+  </xacro:macro>
 </robot>

File: taurob_tracker_description/urdf/tracker_arm_collision_geoms.urdf.xacro (robot description, xacro)
@@ -1,36 +1,35 @@
 <?xml version="1.0"?>
-<robot
-  xmlns:xacro="http://playerstage.sourceforge.net/gazebo/xmlschema/#interface">
-<xacro:macro name="arm_link_0_collision_geom_marco">
-            <collision>
-                <origin xyz="0.0 0.0 0.0" rpy="0 0 0" />
-                <geometry>
-                    <mesh filename="package://taurob_arm_description/meshes/tarm_link_0.stl"/>
-                </geometry>
-            </collision>
-</xacro:macro>
-<xacro:macro name="arm_link_1_collision_geom_marco">
-            <collision>
-                <origin xyz="0.0 0.0 0.0" rpy="0 0 0" />
-                <geometry>
-                    <mesh filename="package://taurob_arm_description/meshes/tarm_link_1.stl"/>
-                </geometry>
-            </collision>
-</xacro:macro>
-<xacro:macro name="arm_link_2_collision_geom_marco">
-            <collision>
-                <origin xyz="0.0 0.0 0.0" rpy="0 0 0" />
-                <geometry>
-                    <mesh filename="package://taurob_arm_description/meshes/tarm_link_2.stl"/>
-                </geometry>
-            </collision>
-</xacro:macro>
-<xacro:macro name="arm_link_3_collision_geom_marco">
-            <collision>
-                <origin xyz="0.0 0.0 0.0" rpy="0 0 0" />
-                <geometry>
-                    <mesh filename="package://taurob_arm_description/meshes/tarm_link_3.stl"/>
-                </geometry>
-            </collision>
-</xacro:macro>
+<robot xmlns:xacro="http://www.ros.org/wiki/xacro">
+  <xacro:macro name="arm_link_0_collision_geom_marco">
+    <collision>
+      <origin xyz="0.0 0.0 0.0" rpy="0 0 0"/>
+      <geometry>
+        <mesh filename="package://taurob_tracker_description/meshes/tarm_link_0.stl"/>
+      </geometry>
+    </collision>
+  </xacro:macro>
+  <xacro:macro name="arm_link_1_collision_geom_marco">
+    <collision>
+      <origin xyz="0.0 0.0 0.0" rpy="0 0 0"/>
+      <geometry>
+        <mesh filename="package://taurob_tracker_description/meshes/tarm_link_1.stl"/>
+      </geometry>
+    </collision>
+  </xacro:macro>
+  <xacro:macro name="arm_link_2_collision_geom_marco">
+    <collision>
+      <origin xyz="0.0 0.0 0.0" rpy="0 0 0"/>
+      <geometry>
+        <mesh filename="package://taurob_tracker_description/meshes/tarm_link_2.stl"/>
+      </geometry>
+    </collision>
+  </xacro:macro>
+  <xacro:macro name="arm_link_3_collision_geom_marco">
+    <collision>
+      <origin xyz="0.0 0.0 0.0" rpy="0 0 0"/>
+      <geometry>
+        <mesh filename="package://taurob_tracker_description/meshes/tarm_link_3.stl"/>
+      </geometry>
+    </collision>
+  </xacro:macro>
 </robot>

File: taurob_tracker_description/urdf/tracker_arm_collision_geoms_simple.urdf.xacro (robot description, xacro)
@@ -3,7 +3,7 @@
   <xacro:macro name="arm_link_0_collision_geom_marco">
     <collision>
-      <origin xyz="0.0 0.0 ${0.137*0.5}" rpy="0 0 0" />
+      <origin xyz="0.0 0.0 ${0.137*0.5}" rpy="0 0 0"/>
       <geometry>
-        <box size="0.08 0.08 0.137" />
+        <box size="0.08 0.08 0.137"/>
       </geometry>
     </collision>
@@ -11,7 +11,7 @@
   <xacro:macro name="arm_link_1_collision_geom_marco">
     <collision>
-      <origin xyz="-0.045 0.18 0.0" rpy="0 0 0" />
+      <origin xyz="-0.045 0.18 0.0" rpy="0 0 0"/>
       <geometry>
-        <box size="0.073 0.4 0.086" />
+        <box size="0.073 0.4 0.086"/>
       </geometry>
     </collision>
@@ -19,7 +19,7 @@
   <xacro:macro name="arm_link_2_collision_geom_marco">
     <collision>
-      <origin xyz="${-0.073*0.5} 0.28 0.0" rpy="0 0 0" />
+      <origin xyz="${-0.073*0.5} 0.28 0.0" rpy="0 0 0"/>
       <geometry>
-        <box size="0.073 0.6 0.086" />
+        <box size="0.073 0.6 0.086"/>
       </geometry>
     </collision>
@@ -27,7 +27,7 @@
   <xacro:macro name="arm_link_3_collision_geom_marco">
     <collision>
-      <origin xyz="0.1 0.05 0.08" rpy="0 0 0" />
+      <origin xyz="0.1 0.05 0.08" rpy="0 0 0"/>
       <geometry>
-        <box size="0.1 0.2 0.18" />
+        <box size="0.1 0.2 0.18"/>
       </geometry>
     </collision>

File: taurob_tracker_description/urdf/tracker_chassis.urdf.xacro (robot description, xacro)
@@ -1,4 +1,4 @@
 <?xml version="1.0"?>
-<robot name="taurob_tracker" xmlns:xacro="http://www.ros.org/wiki/xacro">
+<robot xmlns:xacro="http://www.ros.org/wiki/xacro" name="taurob_tracker">
   <xacro:include filename="$(find hector_xacro_tools)/urdf/inertia_tensors.urdf.xacro"/>
   <xacro:property name="base_size_x" value="${0.365*2}"/>
@@ -17,14 +17,14 @@
       <origin xyz="0 0 0" rpy="0 0 0"/>
       <collision>
-         <origin xyz="0.5 -0.23 ${base_offset_z}" rpy="0 0 0"/>
-         <geometry>
-           <box size="1.05 0.14 0.35"/>
-         </geometry>
+        <origin xyz="0.5 -0.23 ${base_offset_z}" rpy="0 0 0"/>
+        <geometry>
+          <box size="1.05 0.14 0.35"/>
+        </geometry>
       </collision>
       <collision>
-         <origin xyz="0.5 0.23 ${base_offset_z}" rpy="0 0 0"/>
-         <geometry>
-           <box size="1.05 0.14 0.35"/>
-         </geometry>
+        <origin xyz="0.5 0.23 ${base_offset_z}" rpy="0 0 0"/>
+        <geometry>
+          <box size="1.05 0.14 0.35"/>
+        </geometry>
       </collision>
     </link>
@@ -32,10 +32,6 @@
       <origin xyz="${base_offset_x-0.5} 0 0" rpy="0 0 0"/>
       <axis xyz="0 -1 0"/>
-      <limit lower="${-30 * M_PI / 180}" upper="${50 * M_PI / 180}"
-             effort="204" velocity="${1.0 * 110 * M_PI / 180}"/>
-      <safety_controller soft_lower_limit="${-25 * M_PI / 180}"
-                         soft_upper_limit="${45 * M_PI / 180}"
-                         k_position="${100}"
-                         k_velocity="${2}"/>
+      <limit lower="${-30 * M_PI / 180}" upper="${50 * M_PI / 180}" effort="204" velocity="${1.0 * 110 * M_PI / 180}"/>
+      <safety_controller soft_lower_limit="${-25 * M_PI / 180}" soft_upper_limit="${45 * M_PI / 180}" k_position="${100}" k_velocity="${2}"/>
       <parent link="chassis_link"/>
       <child link="flipper_link"/>
@@ -46,7 +42,7 @@
       </xacro:inertial_cuboid_with_pose>
       <visual>
-        <origin xyz="0.0 0.0 0.0" rpy="0 0 0" />
+        <origin xyz="0.0 0.0 0.0" rpy="0 0 0"/>
         <geometry>
-          <mesh filename="package://taurob_tracker_description/meshes/tracker/tracker_chassis.dae"/>
+          <mesh filename="package://taurob_tracker_description/meshes/tracker_chassis.dae"/>
         </geometry>
       </visual>
@@ -66,5 +62,5 @@
         <origin xyz="${base_offset_x} 0.23 ${base_offset_z}" rpy="0 0 0"/>
         <geometry>
-           <box size="1.0 0.13 0.35"/>
+          <box size="1.0 0.13 0.35"/>
         </geometry>
       </collision>
