Commit message: Increase limits for joint 2.

File: taurob_tracker_description/urdf/tracker_arm.urdf.xacro (robot description, xacro)
@@ -65,5 +65,5 @@
       <origin xyz="0.003 0.55 0.03" rpy=" 0 0 0"/>
       <axis xyz="-1 0 0"/>
-      <limit lower="${0 * M_PI / 180}" upper="${180 * M_PI / 180}" effort="1000" velocity="${1.0 * 110 * M_PI / 180}"/>
+      <limit lower="${0}" upper="${2 * M_PI}" effort="1000" velocity="${1.0 * 110 * M_PI / 180}"/>
       <!--        <safety_controller soft_lower_limit="${-168 * M_PI / 180}"
 				 soft_upper_limit="${168 * M_PI / 180}"
